Commit message: "added gazebo simulation and controllers, eps effort controllers"

File: convey_crane_description/convey_crane/robot.urdf.xacro (robot description, xacro)
@@ -1,3 +1,5 @@
-<robot name="convey_crane">
+<?xml version="1.0"?>
+<robot name="convey_crane" xmlns:xacro="http://wiki.ros.org/xacro">
+<xacro:include filename="$(find convey_crane_description)/convey_crane/ros2_control.urdf.xacro"/>
 <link name="support_plaform_1">
 <visual>
@@ -148,5 +150,5 @@
 <joint_properties friction="0.0"/>
 </joint>
-<joint name="continuous_revolute 1" type="continuous">
+<joint name="continuous_revolute_1" type="continuous">
 <origin xyz="0.10468245836551856587 0.024999999999999744649 0" rpy="-0 1.570796326794896336 0" />
 <parent link="cart_move" />
@@ -156,5 +158,5 @@
 <joint_properties friction="0.0"/>
 </joint>
-<joint name="slider 1" type="prismatic">
+<joint name="slider_1" type="prismatic">
 <origin xyz="-0.99499999999999999556 -0.024999999999999966693 -0.039999999999999980016" rpy="-0 -1.570796326794896558 0" />
 <parent link="cart_pole_line" />
